File: mirror_and_rotate.kicad_pcb (KiCad board)
At the start: 6 copper layers, 86.4 x 54.6 mm, 8 parts, among them IC9 TDA19988BHN/C1,557

Commit message: layer change exp
Parts:
- removed IC9 (x7): TDA19988BHN/C1,557, SOT804-4(NXP)
- added IC91: TDA19988BHN/C1,557, SOT804-4(NXP), B.Cu at (110.5, 101.4)
- added IC92: TDA19988BHN/C1,557, SOT804-4(NXP), B.Cu at (110.7, 90.2)
- added IC93: TDA19988BHN/C1,557, SOT804-4(NXP), B.Cu at (110.5, 78.3)
- added IC94: TDA19988BHN/C1,557, SOT804-4(NXP), F.Cu at (123.4, 101.1)
- added IC95: TDA19988BHN/C1,557, SOT804-4(NXP), F.Cu at (123.7, 89.7)
- added IC96: TDA19988BHN/C1,557, SOT804-4(NXP), F.Cu at (123.2, 78.0)
- added IC97: TDA19988BHN/C1,557, SOT804-4(NXP), B.Cu at (110.5, 66.0)
- renumbered IC9 to IC98
Changed lines of the file:
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@@
   (module "SOT804-4(NXP)" (layer Bottom)
     (at 110.4751 101.3766 180)
-    (fp_text reference IC9 (at -4.55 5 90) (layer B.SilkS)
+    (fp_text reference IC91 (at -4.55 5 90) (layer B.SilkS)
       (effects (font (size 0.77216 0.77216) (thickness 0.115824)) (justify right bottom mirror))
     )
@@
   (module "SOT804-4(NXP)" (layer Bottom)
     (at 110.7291 90.2006 270)
-    (fp_text reference IC9 (at -4.55 5) (layer B.SilkS)
+    (fp_text reference IC92 (at -4.55 5) (layer B.SilkS)
       (effects (font (size 0.77216 0.77216) (thickness 0.115824)) (justify left bottom mirror))
     )
@@
   (module "SOT804-4(NXP)" (layer Bottom)
     (at 110.4751 78.2626 90)
-    (fp_text reference IC9 (at -4.55 5) (layer B.SilkS)
+    (fp_text reference IC93 (at -4.55 5) (layer B.SilkS)
       (effects (font (size 0.77216 0.77216) (thickness 0.115824)) (justify right bottom mirror))
     )
@@
   (module "SOT804-4(NXP)" (layer Top)
     (at 123.4291 101.1226 180)
-    (fp_text reference IC9 (at -4.55 -5 90) (layer F.SilkS)
+    (fp_text reference IC94 (at -4.55 -5 90) (layer F.SilkS)
       (effects (font (size 0.77216 0.77216) (thickness 0.115824)) (justify right bottom))
     )
@@
   (module "SOT804-4(NXP)" (layer Top)
     (at 123.6831 89.6926 270)
-    (fp_text reference IC9 (at -4.55 -5) (layer F.SilkS)
+    (fp_text reference IC95 (at -4.55 -5) (layer F.SilkS)
       (effects (font (size 0.77216 0.77216) (thickness 0.115824)) (justify left bottom))
     )
@@
   (module "SOT804-4(NXP)" (layer Top)
     (at 123.1751 78.0086 90)
-    (fp_text reference IC9 (at -4.55 -5) (layer F.SilkS)
+    (fp_text reference IC96 (at -4.55 -5) (layer F.SilkS)
       (effects (font (size 0.77216 0.77216) (thickness 0.115824)) (justify right bottom))
     )
@@
   (module "SOT804-4(NXP)" (layer Bottom)
     (at 110.49 66.04)
-    (fp_text reference IC9 (at -4.55 5 90) (layer B.SilkS)
+    (fp_text reference IC97 (at -4.55 5 90) (layer B.SilkS)
       (effects (font (size 0.77216 0.77216) (thickness 0.115824)) (justify left bottom mirror))
     )
@@
   (module "SOT804-4(NXP)" (layer Top)
     (at 123.19 66.04)
-    (fp_text reference IC9 (at -4.55 -5 -270) (layer F.SilkS)
+    (fp_text reference IC98 (at -4.55 -5 -270) (layer F.SilkS)
       (effects (font (size 0.77216 0.77216) (thickness 0.115824)) (justify left bottom))
     )
